Commit message: Add support for mecanum_controller with omnibot

File: dyno_description/urdf/base/omnibot_base.gazebo.xacro (robot description, xacro)
@@ -11,9 +11,9 @@
   <gazebo>
     <plugin name="object_controller" filename="libgazebo_ros_planar_move.so">
-      <commandTopic>cmd_vel</commandTopic>
-      <odometryTopic>/odom</odometryTopic>
+      <commandTopic>mobile_base_controller/cmd_vel</commandTopic>
+      <odometryTopic>/ground_truth_odom</odometryTopic>
       <odometryFrame>odom</odometryFrame>
       <odometryRate>20.0</odometryRate>
-      <robotBaseFrame>base_footprint</robotBaseFrame>
+      <robotBaseFrame>ground_truth_frame</robotBaseFrame>
     </plugin>
 <!--

File: dyno_description/urdf/base/omnibot_base.urdf.xacro (robot description, xacro)
@@ -18,7 +18,7 @@
       </visual>
       <collision>
-        <origin xyz="0 0 0.04" rpy="0 0 0"/>
+        <origin xyz="0 0 0.02" rpy="0 0 0"/>
         <geometry>
-          <box size="0.4 0.4 0.15"/>
+          <box size="0.42 0.4 0.10"/>
         </geometry>
         <material name="orange"/>
@@ -50,8 +50,8 @@
     <xacro:property name="wheel_torque"     value="6.0"/>
     <xacro:property name="wheel_velocity"   value="1.0"/>
-    <mecanum_wheel name="wheel_front_right"  separation="${wheel_separation}" x_offset="${wheel_separation/2}" reflect="1.0" parent="base_link"/>
-    <mecanum_wheel name="wheel_front_left"   separation="${wheel_separation}" x_offset="${wheel_separation/2}" reflect="-1.0" parent="base_link"/>
-    <mecanum_wheel name="wheel_rear_right"   separation="${wheel_separation}" x_offset="${-wheel_separation/2}" reflect="1.0" parent="base_link"/>
-    <mecanum_wheel name="wheel_rear_left"    separation="${wheel_separation}" x_offset="${-wheel_separation/2}" reflect="-1.0" parent="base_link"/>
+    <mecanum_wheel name="wheel_front_right"  separation="${wheel_separation}" x_offset="${wheel_separation/2}" reflect="1.0" type="right" parent="base_link"/>
+    <mecanum_wheel name="wheel_front_left"   separation="${wheel_separation}" x_offset="${wheel_separation/2}" reflect="-1.0" type="left" parent="base_link"/>
+    <mecanum_wheel name="wheel_rear_right"   separation="${wheel_separation}" x_offset="${-wheel_separation/2}" reflect="1.0" type="left" parent="base_link"/>
+    <mecanum_wheel name="wheel_rear_left"    separation="${wheel_separation}" x_offset="${-wheel_separation/2}" reflect="-1.0" type="right" parent="base_link"/>
     <!-- Gazebo extentions -->
     <base_gazebo/>

File: dyno_description/urdf/wheels/omnibot/mecanum_wheel.urdf.xacro (robot description, xacro)
@@ -3,10 +3,15 @@
   <xacro:include filename="mecanum_wheel.gazebo.xacro"/>
   <xacro:include filename="mecanum_wheel.transmission.xacro"/>
-  <xacro:macro name="mecanum_wheel" params="name separation x_offset reflect parent">
+  <xacro:macro name="mecanum_wheel" params="name separation x_offset reflect type parent">
     <link name="${name}_link">
       <visual>
         <origin xyz="0 0 0" rpy="0 0 0"/>
         <geometry>
-          <mesh filename="package://dyno_description/meshes/mecanum_wheel.stl" scale="0.001 0.001 0.001"/>
+          <xacro:if value="${type == 'left'}">
+            <mesh filename="package://dyno_description/meshes/mecanum_wheel.stl" scale="0.001 0.001 0.001"/>
+          </xacro:if>
+          <xacro:if value="${type == 'right'}">
+            <mesh filename="package://dyno_description/meshes/mecanum_wheel.stl" scale="0.001 0.001 -0.001"/>
+          </xacro:if>
         </geometry>
         <material name="grey"/>
@@ -15,5 +20,5 @@
         <origin xyz="0 0 0" rpy="0 0 0"/>
         <geometry>
-          <cylinder radius="0.1" length="0.05"/>
+          <cylinder radius="0.05" length="0.05"/>
         </geometry>
         <material name="orange"/>
@@ -29,5 +34,5 @@
     </link>
     <joint name="${name}_joint" type="continuous">
-      <origin xyz="${x_offset} ${-separation / 2 * reflect} 0" rpy="${-pi/2} 0 0"/>
+      <origin xyz="${x_offset} ${-separation / 2 * reflect} 0" rpy="${-M_PI/2} 0 0"/>
       <parent link="${parent}"/>
       <child link="${name}_link"/>
