Commit message: Add forklift teb navigation

File: dyno_description/urdf/base/forklift_base.urdf.xacro (robot description, xacro)
@@ -22,8 +22,9 @@
         <material name="orange"/>
       </collision>
+      <!-- Set high weight and low intertia for gazebot simulation -->
       <inertial>
-        <origin xyz="0.1 0 0" rpy="0 0 0"/>
-        <mass value="1.0"/>
-        <box_inertia m="1.0" x="0.3" y="0.25" z="0.1"/>
+        <origin xyz="0.13 0 0" rpy="0 0 0"/>
+        <mass value="10.0"/>
+        <box_inertia m="0.1" x="0.3" y="0.25" z="0.1"/>
       </inertial>
     </link>
@@ -31,5 +32,5 @@
     <link name="base_footprint"/>
     <joint name="base_footprint_joint" type="fixed">
-      <origin xyz="0 0 0.25" rpy="0 0 0"/>
+      <origin xyz="0 0 0.025" rpy="0 0 0"/>
       <parent link="base_footprint"/>
       <child link="base_link"/>
@@ -60,6 +61,6 @@
       <inertial>
         <origin xyz="-0.16 0 0" rpy="0 0 0"/>
-        <mass value="0.2"/>
-        <box_inertia m="0.2" x="0.23" y="0.1" z="0.008"/>
+        <mass value="0.02"/>
+        <box_inertia m="0.002" x="0.23" y="0.1" z="0.008"/>
       </inertial>
     </link>

File: dyno_description/urdf/wheels/forklift/drive_wheel_assembly.urdf.xacro (robot description, xacro)
@@ -19,4 +19,7 @@
       <child link="drive_wheel_link"/>
     </joint>
+    <xacro:if value="$(arg use_ros_control_for_base)">
+      <xacro:simple_transmission name="drive_wheel_joint" interface="VelocityJointInterface"/>
+    </xacro:if>
     <link name="drive_wheel_link">
       <inertial>

File: dyno_description/urdf/wheels/forklift/support_wheel.gazebo.xacro (robot description, xacro)
@@ -6,6 +6,6 @@
      <kp>100000.0</kp>
      <kd>100.0</kd>
-     <mu1>1.0</mu1>
-     <mu2>1.0</mu2>
+     <mu1>100.0</mu1>
+     <!-- <mu2>1.0</mu2> -->
      <fdir1>1 0 0</fdir1>
      <maxVel>1.0</maxVel>

File: dyno_description/urdf/wheels/forklift/support_wheel.urdf.xacro (robot description, xacro)
@@ -36,5 +36,5 @@
     <!-- Transmission -->
     <xacro:if value="$(arg use_ros_control_for_base)">
-      <xacro:simple_transmission name="${suffix}_steer_joint" interface="VelocityJointInterface"/>
+      <xacro:simple_transmission name="${name}_joint" interface="EffortJointInterface"/>
     </xacro:if>
     <!-- Gazebo extensions -->

Commit message: Change fork z origin

File: dyno_description/urdf/base/forklift_base.urdf.xacro (robot description, xacro)
@@ -38,5 +38,5 @@
     <!-- Fork -->
     <joint name="fork_joint" type="prismatic">
-      <origin xyz="0.106 0 0" rpy="0 0 0"/>
+      <origin xyz="0.106 0 -0.013" rpy="0 0 0"/>
       <parent link="base_link"/>
       <child link="fork_link"/>
