Commit message: Add fake vive localization

File: dyno_description/urdf/base/magni_sign_base.gazebo.xacro (robot description, xacro)
@@ -6,5 +6,5 @@
     </gazebo>
     <gazebo reference="sign_pole_link">
-      <material>Gazebo/DarkGrey</material>
+      <material>Gazebo/Grey</material>
     </gazebo>
     <gazebo reference="base_footprint">

File: dyno_description/urdf/base/magni_sign_base.urdf.xacro (robot description, xacro)
@@ -54,5 +54,5 @@
           <mesh filename="package://dyno_description/meshes/other/sign_pole.stl" scale="0.01 0.01 0.01"/>
         </geometry>
-        <material name="black"/>
+        <material name="grey"/>
       </visual>
     </link>

File: dyno_description/urdf/sensors/sick_tim.urdf.xacro (robot description, xacro)
@@ -23,8 +23,8 @@
     <joint name="${name}_joint" type="fixed">
       <parent link="${name}_mount_link" />
-      <child link="${name}" />
+      <child link="${name}_link" />
       <origin rpy="0 0 0" xyz="0 0 ${z_offset}"/>
     </joint>
-    <link name="${name}">
+    <link name="${name}_link">
       <visual>
         <geometry>
