Commit message: Add navigation to multiple platforms

File: dyno_description/robots/holonomic.xacro (robot description, xacro)
@@ -12,5 +12,5 @@
   <base/>
   <!-- Laser Scanner -->
-  <lds_lfcd name="base_scan" x_offset="0" y_offset="0" z_offset="0.17" yaw_offset="0" parent="base_link"/>
+  <lds_lfcd name="base_scan" x_offset="0" y_offset="0" z_offset="0.175" yaw_offset="0" parent="base_link"/>
   <!-- Imu -->
   <imu x_offset="0" y_offset="0" z_offset="0"/>

File: dyno_description/urdf/base/magni_base.urdf.xacro (robot description, xacro)
@@ -12,5 +12,5 @@
   <xacro:property name="wheel_velocity"   value="1.0"/>
   <!-- Caster characteristics -->
-  <xacro:property name="caster_radius" value="0.05"/>
+  <xacro:property name="caster_radius" value="0.04"/>
   <xacro:property name="caster_ground_offset" value="0.005"/>
   <!-- Base -->

File: dyno_description/urdf/base/omnibot_base.gazebo.xacro (robot description, xacro)
@@ -6,5 +6,7 @@
     </gazebo>
     <gazebo reference="base_footprint">
+      <!--
       <kinematic>true</kinematic>
+      -->
     </gazebo>
     <gazebo>

File: dyno_description/urdf/base/turtlebot3_burger.urdf.xacro (robot description, xacro)
@@ -27,5 +27,5 @@
       </collision>
       <inertial>
-        <origin xyz="0 0 0" rpy="0 0 0"/>
+        <origin xyz="-0.03 0 0" rpy="0 0 0"/>
         <mass value="8.2573504e-01"/>
         <inertia ixx="2.2124416e-03" ixy="-1.2294101e-05" ixz="3.4938785e-05"

File: dyno_description/urdf/wheels/turtlebot3/drive_wheel.gazebo.xacro (robot description, xacro)
@@ -5,8 +5,12 @@
   <!-- TEMPORARY: Set friction very low and control base with gazebo planar move -->
   <gazebo reference="${name}_link">
+    <!--
+    <kp>500000.0</kp>
+    <kd>10.0</kd>
+     -->
+    <kp>100000.0</kp>
+    <kd>100.0</kd>
     <mu1>0.1</mu1>
     <mu2>0.1</mu2>
-    <kp>500000.0</kp>
-    <kd>10.0</kd>
     <minDepth>0.001</minDepth>
     <maxVel>0.1</maxVel>
