Commit message: Fix colors in leap_motion collada mesh and rotate

File: dyno_description/robots/forklift.xacro (robot description, xacro)
@@ -18,5 +18,5 @@
   <!-- <vive_tracker name="vive_tracker" x_offset="0.13" y_offset="0" z_offset="0.391" yaw_offset="0" parent="base_link"/> -->
   <!-- Leap Motion -->
-  <leap_motion name="leap_motion" x_offset="-0.025" y_offset="0" z_offset="0.08" yaw_offset="0" parent="fork_link"/>
+  <leap_motion name="leap_motion" x_offset="-0.024" y_offset="0" z_offset="0.08" yaw_offset="${M_PI}" parent="fork_link"/>
   <!-- Imu -->
   <imu x_offset="0" y_offset="0" z_offset="0"/>

File: dyno_description/urdf/sensors/leap_motion.gazebo.xacro (robot description, xacro)
@@ -3,5 +3,5 @@
   <xacro:macro name="leap_motion_gazebo" params="name">
     <gazebo reference="${name}_link">
-      <material>Gazebo/Grey</material>
+      <!-- <material>Gazebo/Grey</material> -->
     </gazebo>
   </xacro:macro>

File: dyno_description/urdf/sensors/leap_motion.urdf.xacro (robot description, xacro)
@@ -12,5 +12,5 @@
         <origin xyz="0 0 0.0" rpy="0 0 0"/>
         <geometry>
-          <mesh filename="package://dyno_description/meshes/sensors/leap_motion.stl" scale="0.01 0.01 0.01"/>
+          <mesh filename="package://dyno_description/meshes/sensors/leap_motion.dae" scale="0.01 0.01 0.01"/>
         </geometry>
         <material name="grey"/>
