Commit message: Add open manipulator to omnibot (dependecy on robotis)

File: dyno_description/robots/omnibot.xacro (robot description, xacro)
@@ -9,9 +9,11 @@
   <xacro:include filename="../urdf/sensors/lds_lfcd.urdf.xacro"/>
   <xacro:include filename="../urdf/sensors/imu.urdf.xacro"/>
+  <xacro:include filename="../urdf/manipulators/open_manipulator.urdf.xacro"/>
   <!-- Use macros to define the actual robot -->
   <base/>
   <!-- Laser Scanner -->
-  <lds_lfcd name="base_scan" x_offset="0" y_offset="0" z_offset="0.1" yaw_offset="0" parent="base_link"/>
+  <lds_lfcd name="base_scan" x_offset="0.15" y_offset="0" z_offset="0.1" yaw_offset="0" parent="base_link"/>
   <!-- Imu -->
   <imu x_offset="0" y_offset="0" z_offset="0"/>
+  <open_manipulator x_offset="0.08" y_offset="0" z_offset="0.07"/>
 </robot>

File: dyno_description/urdf/sensors/leap_motion.gazebo.xacro (robot description, xacro)
@@ -3,5 +3,5 @@
   <xacro:macro name="leap_motion_gazebo" params="name">
     <gazebo reference="${name}_link">
-      <!-- <material>Gazebo/Grey</material> -->
+      <material>Gazebo/Grey</material>
     </gazebo>
   </xacro:macro>

File: dyno_description/urdf/sensors/leap_motion.urdf.xacro (robot description, xacro)
@@ -12,5 +12,5 @@
         <origin xyz="0 0 0.0" rpy="0 0 0"/>
         <geometry>
-          <mesh filename="package://dyno_description/meshes/sensors/leap_motion.dae" scale="0.01 0.01 0.01"/>
+          <mesh filename="package://dyno_description/meshes/sensors/leap_motion.stl" scale="0.01 0.01 0.01"/>
         </geometry>
         <material name="grey"/>
