Commit message: Remove open manipulator dependency

File: dyno_description/robots/diff_drive.xacro (robot description, xacro)
@@ -1,4 +1,5 @@
 <?xml version="1.0"?>
 <robot xmlns:xacro="http://ros.org/wiki/xacro" name="dyno_diff_drive" >
+  <xacro:arg name="use_ros_control_for_base" default="true"/>
   <xacro:include filename="../urdf/materials/materials.xacro"/>
   <xacro:include filename="../urdf/utils.urdf.xacro"/>
@@ -7,5 +8,5 @@
   <xacro:include filename="../urdf/base/diff_drive_base.urdf.xacro"/>
   <xacro:include filename="../urdf/sensors/lds_lfcd.urdf.xacro"/>
-  <xacro:include filename="../urdf/sensors/imu.urdf.xacro"/>
+  <!-- <xacro:include filename="../urdf/sensors/imu.urdf.xacro"/> -->
   <!-- Use macros to define the actual robot -->
   <base/>
@@ -13,4 +14,4 @@
   <lds_lfcd name="base_scan" x_offset="0" y_offset="0" z_offset="0.17" yaw_offset="0" parent="base_link"/>
   <!-- Imu -->
-  <imu x_offset="0" y_offset="0" z_offset="0"/>
+  <!-- <imu x_offset="0" y_offset="0" z_offset="0"/> -->
 </robot>

File: dyno_description/urdf/base/omnibot_base.urdf.xacro (robot description, xacro)
@@ -15,5 +15,5 @@
           <mesh filename="package://dyno_description/meshes/bases/omnibot_base.stl" scale="0.001 0.001 0.001"/>
         </geometry>
-        <material name="blue"/>
+        <material name="light_blue"/>
       </visual>
       <collision>

File: dyno_description/urdf/manipulators/open_manipulator.urdf.xacro (robot description, xacro)
@@ -3,5 +3,5 @@
 <robot xmlns:xacro="http://www.ros.org/wiki/xacro">
   <!-- Include OpenManipulator Chain Gazebo Parameter -->
-  <xacro:include filename="$(find open_manipulator_with_tb3_description)/urdf/open_manipulator_with_tb3.gazebo.xacro"/>
+  <xacro:include filename="$(find dyno_description)/urdf/manipulators/open_manipulator.gazebo.xacro"/>
   <xacro:macro name="open_manipulator" params="x_offset y_offset z_offset">
     <!-- Base fixed joint -->
@@ -16,12 +16,12 @@
         <origin xyz="0 0 0" rpy="0 0 0"/>
         <geometry>
-          <mesh filename="package://open_manipulator_with_tb3_description/meshes/chain_link1.stl" scale="0.001 0.001 0.001"/>
-        </geometry>
-        <material name="grey"/>
-      </visual>
-      <collision>
-        <origin xyz="0 0 0" rpy="0 0 0"/>
-        <geometry>
-          <mesh filename="package://open_manipulator_with_tb3_description/meshes/chain_link1.stl" scale="0.001 0.001 0.001"/>
+          <mesh filename="package://dyno_description/meshes/manipulators/open_manipulator/chain_link1.stl" scale="0.001 0.001 0.001"/>
+        </geometry>
+        <material name="dark"/>
+      </visual>
+      <collision>
+        <origin xyz="0 0 0" rpy="0 0 0"/>
+        <geometry>
+          <mesh filename="package://dyno_description/meshes/manipulators/open_manipulator/chain_link1.stl" scale="0.001 0.001 0.001"/>
         </geometry>
       </collision>
@@ -57,12 +57,12 @@
         <origin xyz="0 0 0.018" rpy="0 0 0"/>
         <geometry>
-          <mesh filename="package://open_manipulator_with_tb3_description/meshes/chain_link2.stl" scale="0.001 0.001 0.001"/>
-        </geometry>
-        <material name="grey"/>
+          <mesh filename="package://dyno_description/meshes/manipulators/open_manipulator/chain_link2.stl" scale="0.001 0.001 0.001"/>
+        </geometry>
+        <material name="dark"/>
       </visual>
       <collision>
         <origin xyz="0 0 0.018" rpy="0 0 0"/>
         <geometry>
-          <mesh filename="package://open_manipulator_with_tb3_description/meshes/chain_link2.stl" scale="0.001 0.001 0.001"/>
+          <mesh filename="package://dyno_description/meshes/manipulators/open_manipulator/chain_link2.stl" scale="0.001 0.001 0.001"/>
         </geometry>
       </collision>
@@ -99,12 +99,12 @@
         <origin xyz="0 0 0" rpy="0 0 0"/>
         <geometry>
-          <mesh filename="package://open_manipulator_with_tb3_description/meshes/chain_link3.stl" scale="0.001 0.001 0.001"/>
-        </geometry>
-        <material name="grey"/>
-      </visual>
-      <collision>
-        <origin xyz="0 0 0" rpy="0 0 0"/>
-        <geometry>
-          <mesh filename="package://open_manipulator_with_tb3_description/meshes/chain_link3.stl" scale="0.001 0.001 0.001"/>
+          <mesh filename="package://dyno_description/meshes/manipulators/open_manipulator/chain_link3.stl" scale="0.001 0.001 0.001"/>
+        </geometry>
+        <material name="dark"/>
+      </visual>
+      <collision>
+        <origin xyz="0 0 0" rpy="0 0 0"/>
+        <geometry>
+          <mesh filename="package://dyno_description/meshes/manipulators/open_manipulator/chain_link3.stl" scale="0.001 0.001 0.001"/>
         </geometry>
       </collision>
@@ -141,12 +141,12 @@
         <origin xyz="0 0 0" rpy="0 0 0"/>
         <geometry>
-          <mesh filename="package://open_manipulator_with_tb3_description/meshes/chain_link4.stl" scale="0.001 0.001 0.001"/>
-        </geometry>
-        <material name="grey"/>
-      </visual>
-      <collision>
-        <origin xyz="0 0 0" rpy="0 0 0"/>
-        <geometry>
-          <mesh filename="package://open_manipulator_with_tb3_description/meshes/chain_link4.stl" scale="0.001 0.001 0.001"/>
+          <mesh filename="package://dyno_description/meshes/manipulators/open_manipulator/chain_link4.stl" scale="0.001 0.001 0.001"/>
+        </geometry>
+        <material name="dark"/>
+      </visual>
+      <collision>
+        <origin xyz="0 0 0" rpy="0 0 0"/>
+        <geometry>
+          <mesh filename="package://dyno_description/meshes/manipulators/open_manipulator/chain_link4.stl" scale="0.001 0.001 0.001"/>
         </geometry>
       </collision>
@@ -183,12 +183,12 @@
         <origin xyz="0 0 0" rpy="0 0 0"/>
         <geometry>
-          <mesh filename="package://open_manipulator_with_tb3_description/meshes/chain_link5.stl" scale="0.001 0.001 0.001"/>
-        </geometry>
-        <material name="grey"/>
-      </visual>
-      <collision>
-        <origin xyz="0 0 0" rpy="0 0 0"/>
-        <geometry>
-          <mesh filename="package://open_manipulator_with_tb3_description/meshes/chain_link5.stl" scale="0.001 0.001 0.001"/>
+          <mesh filename="package://dyno_description/meshes/manipulators/open_manipulator/chain_link5.stl" scale="0.001 0.001 0.001"/>
+        </geometry>
+        <material name="dark"/>
+      </visual>
+      <collision>
+        <origin xyz="0 0 0" rpy="0 0 0"/>
+        <geometry>
+          <mesh filename="package://dyno_description/meshes/manipulators/open_manipulator/chain_link5.stl" scale="0.001 0.001 0.001"/>
         </geometry>
       </collision>
@@ -205,12 +205,12 @@
         <origin xyz="0.028 0.0246 0" rpy="0 0 0"/>
         <geometry>
-          <mesh filename="package://open_manipulator_with_tb3_description/meshes/chain_link_grip_l.stl" scale="0.001 0.001 0.001"/>
-        </geometry>
-        <material name="grey"/>
+          <mesh filename="package://dyno_description/meshes/manipulators/open_manipulator/chain_link_grip_l.stl" scale="0.001 0.001 0.001"/>
+        </geometry>
+        <material name="dark"/>
       </visual>
       <collision>
         <origin xyz="0.028 0.0246 0" rpy="0 0 0"/>
         <geometry>
-          <mesh filename="package://open_manipulator_with_tb3_description/meshes/chain_link_grip_l.stl" scale="0.001 0.001 0.001"/>
+          <mesh filename="package://dyno_description/meshes/manipulators/open_manipulator/chain_link_grip_l.stl" scale="0.001 0.001 0.001"/>
         </geometry>
       </collision>
@@ -247,12 +247,12 @@
         <origin xyz="0.028 -0.0246 0" rpy="0 0 0"/>
         <geometry>
-          <mesh filename="package://open_manipulator_with_tb3_description/meshes/chain_link_grip_r.stl" scale="0.001 0.001 0.001"/>
-        </geometry>
-        <material name="grey"/>
+          <mesh filename="package://dyno_description/meshes/manipulators/open_manipulator/chain_link_grip_r.stl" scale="0.001 0.001 0.001"/>
+        </geometry>
+        <material name="dark"/>
       </visual>
       <collision>
         <origin xyz="0.028 -0.0246 0" rpy="0 0 0"/>
         <geometry>
-          <mesh filename="package://open_manipulator_with_tb3_description/meshes/chain_link_grip_r.stl" scale="0.001 0.001 0.001"/>
+          <mesh filename="package://dyno_description/meshes/manipulators/open_manipulator/chain_link_grip_r.stl" scale="0.001 0.001 0.001"/>
         </geometry>
       </collision>

File: dyno_description/urdf/sensors/imu.urdf.xacro (robot description, xacro)
@@ -3,5 +3,17 @@
   <xacro:include filename="imu.gazebo.xacro"/>
   <xacro:macro name="imu" params="x_offset y_offset z_offset">
-    <link name="imu_link"/>
+    <link name="imu_link">
+      <visual>
+        <origin xyz="0 0 0.0" rpy="0 0 0"/>
+        <geometry>
+          <cylinder length="0.001" radius="0.001"/>
+        </geometry>
+      </visual>
+      <inertial>
+        <origin xyz="0 0 0" rpy="0 0 0"/>
+        <mass value="0.001"/>
+        <box_inertia m="0.001" x="0.01" y="0.01" z="0.002"/>
+      </inertial>
+    </link>
     <joint name="imu_joint" type="fixed">
       <origin xyz="${x_offset} ${y_offset} ${z_offset}" rpy="0 0 0"/>

File: dyno_description/urdf/sensors/lds_lfcd.urdf.xacro (robot description, xacro)
@@ -13,4 +13,5 @@
         <geometry>
           <mesh filename="package://dyno_description/meshes/sensors/lds.stl" scale="0.001 0.001 0.001"/>
+          <!-- <cylinder length="0.0315" radius="0.055"/> -->
         </geometry>
         <material name="dark"/>

File: dyno_description/urdf/sensors/leap_motion.urdf.xacro (robot description, xacro)
@@ -12,7 +12,7 @@
         <origin xyz="0 0 0.0" rpy="0 0 0"/>
         <geometry>
-          <mesh filename="package://dyno_description/meshes/sensors/leap_motion.stl" scale="0.01 0.01 0.01"/>
+          <mesh filename="package://dyno_description/meshes/sensors/leap_motion.dae" scale="0.01 0.01 0.01"/>
         </geometry>
-        <material name="grey"/>
+        <!-- <material name="grey"/> -->
       </visual>
       <!--

File: dyno_description/urdf/wheels/omnibot/mecanum_wheel.urdf.xacro (robot description, xacro)
@@ -15,5 +15,5 @@
           </xacro:if>
         </geometry>
-        <material name="grey"/>
+        <material name="dark"/>
       </visual>
       <collision>

Commit message: Add magni sign base

File: dyno_description/robots/diff_drive.xacro (robot description, xacro)
@@ -2,4 +2,5 @@
 <robot xmlns:xacro="http://ros.org/wiki/xacro" name="dyno_diff_drive" >
   <xacro:arg name="use_ros_control_for_base" default="true"/>
+  <xacro:arg name="base_variant" default="default"/>
   <xacro:include filename="../urdf/materials/materials.xacro"/>
   <xacro:include filename="../urdf/utils.urdf.xacro"/>

File: dyno_description/robots/forklift.xacro (robot description, xacro)
@@ -2,4 +2,5 @@
 <robot xmlns:xacro="http://ros.org/wiki/xacro" name="dyno_forklift" >
   <xacro:arg name="use_ros_control_for_base" default="true"/>
+  <xacro:arg name="base_variant" default="default"/>
   <xacro:include filename="../urdf/materials/materials.xacro"/>
   <xacro:include filename="../urdf/utils.urdf.xacro"/>

File: dyno_description/robots/holonomic.xacro (robot description, xacro)
@@ -2,4 +2,5 @@
 <robot xmlns:xacro="http://ros.org/wiki/xacro" name="dyno_holonomic" >
   <xacro:arg name="use_ros_control_for_base" default="true"/>
+  <xacro:arg name="base_variant" default="default"/>
   <xacro:include filename="../urdf/materials/materials.xacro"/>
   <xacro:include filename="../urdf/utils.urdf.xacro"/>

File: dyno_description/robots/magni.xacro (robot description, xacro)
@@ -2,16 +2,34 @@
 <robot xmlns:xacro="http://ros.org/wiki/xacro" name="dyno_magni" >
   <xacro:arg name="use_ros_control_for_base" default="true"/>
+  <xacro:arg name="base_variant" default="default"/>
+  <xacro:property name="base_variant" value="$(arg base_variant)"/>
   <xacro:include filename="../urdf/materials/materials.xacro"/>
   <xacro:include filename="../urdf/utils.urdf.xacro"/>
   <xacro:include filename="../urdf/plugins.gazebo.xacro"/>
   <!-- Set up definitions of parts of robot body -->
-  <xacro:include filename="../urdf/base/magni_base.urdf.xacro"/>
-  <xacro:include filename="../urdf/sensors/lds_lfcd.urdf.xacro"/>
-  <xacro:include filename="../urdf/sensors/imu.urdf.xacro"/>
-  <!-- Use macros to define the actual robot -->
-  <base/>
-  <!-- Laser Scanner -->
-  <lds_lfcd name="base_scan" x_offset="0" y_offset="0" z_offset="0.2" yaw_offset="0" parent="base_link"/>
-  <!-- Imu -->
-  <imu x_offset="0" y_offset="0" z_offset="0"/>
+  <xacro:if value="${base_variant == 'default'}">
+    <xacro:include filename="../urdf/base/magni_base.urdf.xacro"/>
+    <xacro:include filename="../urdf/sensors/lds_lfcd.urdf.xacro"/>
+    <xacro:include filename="../urdf/sensors/imu.urdf.xacro"/>
+    <!-- Use macros to define the actual robot -->
+    <base/>
+    <!-- Laser Scanner -->
+    <lds_lfcd name="base_scan" x_offset="0" y_offset="0" z_offset="0.2" yaw_offset="0" parent="base_link"/>
+    <!-- Imu -->
+    <imu x_offset="0" y_offset="0" z_offset="0"/>
+  </xacro:if>
+  <xacro:if value="${base_variant == 'sign'}">
+    <xacro:include filename="../urdf/base/magni_sign_base.urdf.xacro"/>
+    <xacro:include filename="../urdf/sensors/sick_tim.urdf.xacro"/>
+    <xacro:include filename="../urdf/sensors/rplidar_a2.urdf.xacro"/>
+    <!-- Use macros to define the actual robot -->
+    <base/>
+    <joint name="base_scan_mount_joint" type="fixed">
+      <origin xyz="0.0725 0 1.85" rpy="0 0 0"/>
+      <child link="base_scan_mount_link"/>
+      <parent link="sign_pole_link"/>
+    </joint>
+    <sick_tim571 name="base_scan" ros_topic="scan"/>
+    <rplidar_a2 name="obstacle_scan" x_offset="0.06" y_offset="0" z_offset="0.11" yaw_offset="0" parent="base_link"/>
+  </xacro:if>
 </robot>

File: dyno_description/robots/omnibot.xacro (robot description, xacro)
@@ -2,4 +2,5 @@
 <robot xmlns:xacro="http://ros.org/wiki/xacro" name="dyno_omnibot" >
   <xacro:arg name="use_ros_control_for_base" default="true"/>
+  <xacro:arg name="base_variant" default="default"/>
   <xacro:include filename="../urdf/materials/materials.xacro"/>
   <xacro:include filename="../urdf/utils.urdf.xacro"/>

File: dyno_description/robots/quadrotor.xacro (robot description, xacro)
@@ -2,4 +2,5 @@
 <robot name="dyno_quadrotor" xmlns:xacro="http://www.ros.org/wiki/xacro">
   <xacro:arg name="use_ros_control_for_base" default="true"/>
+  <xacro:arg name="base_variant" default="default"/>
   <xacro:include filename="../urdf/materials/materials.xacro"/>
   <xacro:include filename="../urdf/utils.urdf.xacro"/>

File: dyno_description/robots/turtlebot3.xacro (robot description, xacro)
@@ -2,4 +2,5 @@
 <robot xmlns:xacro="http://ros.org/wiki/xacro" name="dyno_turtlebot" >
   <xacro:arg name="use_ros_control_for_base" default="true"/>
+  <xacro:arg name="base_variant" default="default"/>
   <xacro:include filename="../urdf/materials/materials.xacro"/>
   <xacro:include filename="../urdf/utils.urdf.xacro"/>

File: dyno_description/urdf/wheels/magni/drive_wheel.urdf.xacro (robot description, xacro)
@@ -8,7 +8,7 @@
         <origin xyz="0 0 0" rpy="0 0 0"/>
         <geometry>
-          <cylinder radius="${radius}" length="${width}"/>
+          <!-- <cylinder radius="${radius}" length="${width}"/> -->
+          <mesh filename="package://dyno_description/meshes/wheels/magni_wheel.dae" scale="0.0118 0.0118 ${-0.0118 * reflect}"/>
         </geometry>
-        <material name="black"/>
       </visual>
       <collision>
