Commit message: Add forklift urdf

File: dyno_description/urdf/materials/materials.xacro (robot description, xacro)
@@ -12,4 +12,7 @@
   <material name="blue">
     <color rgba="0.0 0.0 0.8 1.0"/>
+  </material>
+  <material name="light_blue">
+    <color rgba="0.3 0.3 0.8 1.0"/>
   </material>
   <material name="green">
